File: BuzzerBoard/v2.brd (EAGLE design)
At the start: 48 x 15 mm, 12 parts, among them J1 input, J2 speaker, J3 inv, U2 LM48310SD/NOPBSDA10A-M

Commit message: V2 to oshpark.
Parts:
- moved U$2 2.43 mm to (24.4, 0.60)
- moved C1 1.03 mm to (26.4, 6.55), turned to 180 degrees
- moved C6 0.21 mm to (16.9, 7.10)
- moved C3 0.20 mm to (18.6, 7.10)
- moved C5 0.10 mm to (18.0, 10.7)
Routing:
- net P0: track 0.00 -> 9.80 mm, vias 0 -> 2
- net 3.3V: track 0.00 -> 8.79 mm, vias 0 -> 1
- net +: track 0.00 -> 7.54 mm
- net -: track 0.00 -> 5.58 mm, vias 0 -> 1
- net BAL_IN: track 0.00 -> 4.83 mm
- net GND: track 0.00 -> 3.27 mm, vias 0 -> 4
- net BAL_IN_RAW: track 0.00 -> 2.79 mm
- net P0_RAW: track 0.00 -> 2.73 mm
- added copper zone on layer 1, net 3.3V
- added copper zone on layer 16, net GND
- removed copper zone on layer 1, net N$1
Other:
- board text added: "-"
- board text added: "IN+"
- board text added: "P0/IN-"
- board text removed: "P0"
